File: pcb/probe-adapter/probe-adapter.kicad_pcb (KiCad board)
At the start: 2 copper layers, 18 x 31 mm, 6 parts

Commit message: sync : export gerber
Parts:
- removed the REF** at (181.5, 113.0)
- removed the REF** at (176.5, 113.0)
- removed the REF** at (186.5, 113.0)
- added C1: 10u, Capacitor_SMD:C_0805_2012Metric_Pad1.18x1.45mm_HandSolder, F.Cu at (181.8, 115.0)
- added C2: (OPTIONAL)22-100n, Capacitor_SMD:C_0805_2012Metric_Pad1.18x1.45mm_HandSolder, F.Cu at (181.5, 118.2)
- added D1: WS2812B, LED_SMD:LED_WS2812B_PLCC4_5.0x5.0mm_P3.2mm, F.Cu at (181.5, 109.5)
- added G***: LOGO, custom-footprints:snakeoilxy-text-logo-SM, B.Cu at (181.5, 106.0)
- added J1: NEOPIXEL, custom-footprints:solder-pad, B.Cu at (188.8, 116.0)
- added J2: GND, custom-footprints:solder-pad, B.Cu at (174.2, 116.0)
- added J3: PROBE, custom-footprints:solder-pad, B.Cu at (185.8, 116.0)
- added J4: 5V, custom-footprints:solder-pad, B.Cu at (177.2, 116.0)
- added J5: POGO_MAGNET, custom-footprints:pogo-magnet-2p, F.Cu at (176.5, 113.0)
- added J6: POGO_MAGNET, custom-footprints:pogo-magnet-2p, F.Cu at (186.5, 113.0)
Routing:
- net NEOPIXEL: track 0.00 -> 17.7 mm, vias 0 -> 1
- net PROBE: track 0.00 -> 10.4 mm, vias 0 -> 1
- net 5V: track 0.00 -> 8.99 mm, vias 0 -> 1
- added copper zone on B.Cu, net GND
- added copper zone on F.Cu, net GND
Other:
- board text added: "5V"
- board text added: "GND"
- board text added: "LED"
- board text added: "PROBE"
- board text added: "Probe Adapter"
- board text added: "Rev.1"
